File: mpu.kicad_sch (KiCad schematic)
At the start: 22 parts, among them SW401 SW_DIP_x03, U401 STM32MP135FAE7, Y401 32.768 kHz, Y402 24 MHz

Commit message: Add ETH schema
Parts:
- added R405, R406, R407, R410: 33 Ω, perfect_footprints:R_0402_1005Metric, symbol Device:R
- R402: Tolerance (none) -> ± 1 %
- renumbered R404 to R403, R403 to R404, R405 to R408, R406 to R409, R407 to R411
Connections:
- net BOOT1: now also U401.P12 (PI5); no longer U401.H2 (PI3)
- net BOOT2: now also U401.R12 (PI6); no longer U401.J3 (PI2)
- net LSE_IN: now also U401.K1 (PC14); no longer U401.K1 (PC14)
- net LSE_OUT: now also U401.K2 (PC15); no longer U401.K2 (PC15)
- net ETH.TXD0: now reaches U401.P8 (PG13)
- net ETH.TXD1: now reaches U401.P9 (PG14)
- net ETH.MDC: now reaches U401.R1 (PG2)
- net ETH.TXEN: now reaches U401.N5 (PB11)
- net ETH.MDIO: now reaches U401.P5 (PA2)
- net ETH.REF_CLK: now reaches U401.T2 (PA11)
- net A0 renamed DDR.A0
- net A1 renamed DDR.A1
- net A10 renamed DDR.A10
- net A11 renamed DDR.A11
- net A12 renamed DDR.A12
- net A13 renamed DDR.A13
- net A14 renamed DDR.A14
- net A15 renamed DDR.A15
- net A2 renamed DDR.A2
- net A3 renamed DDR.A3
- net A4 renamed DDR.A4
- net A5 renamed DDR.A5
- net A6 renamed DDR.A6
- net A7 renamed DDR.A7
- net A8 renamed DDR.A8
- net A9 renamed DDR.A9
- net BA0 renamed DDR.BA0
- net BA1 renamed DDR.BA1
- net BA2 renamed DDR.BA2
- net CAS_N renamed DDR.CAS_N
- net CKE renamed DDR.CKE
- net CLK_N renamed DDR.CLK_N
- net CLK_P renamed DDR.CLK_P
- net CS_N renamed DDR.CS_N
- net CTRL renamed PMIC.CTRL
- net DQ0 renamed DDR.DQ0
- net DQ1 renamed DDR.DQ1
- net DQ10 renamed DDR.DQ10
- net DQ11 renamed DDR.DQ11
- net DQ12 renamed DDR.DQ12
- net DQ13 renamed DDR.DQ13
- net DQ14 renamed DDR.DQ14
- net DQ15 renamed DDR.DQ15
- net DQ2 renamed DDR.DQ2
- net DQ3 renamed DDR.DQ3
- net DQ4 renamed DDR.DQ4
- net DQ5 renamed DDR.DQ5
- net DQ6 renamed DDR.DQ6
- net DQ7 renamed DDR.DQ7
- net DQ8 renamed DDR.DQ8
- net DQ9 renamed DDR.DQ9
- net DQM0 renamed DDR.DQM0
- net DQM1 renamed DDR.DQM1
- net DQS_N0 renamed DDR.DQS0_N
- net DQS_N1 renamed DDR.DQS1_N
- net DQS_P0 renamed DDR.DQS0_P
- net DQS_P1 renamed DDR.DQS1_P
- removed net INT_N: U401.G5 (PF8)
- net JTCK renamed JTAG.JTCK
- net JTDI renamed JTAG.JTDI
- net JTDO renamed JTAG.JTDO
- net JTMS renamed JTAG.JTMS
- net JTRST_N renamed JTAG.JTRST_N
- net ODT renamed DDR.ODT
- net RAS_N renamed DDR.RAS_N
- net RST_N renamed PMIC.RST_N
- net PMIC.RST_N: no longer U401.E17 (DDR_RESETN)
- net RX renamed DEBUG.RX
- net DEBUG.RX: now also U401.C5 (PD8); no longer U401.C5 (PD8)
- removed net SCL: U401.D8 (PE15)
- net SDA renamed PMIC.SDA
- net TX renamed DEBUG.TX
- net DEBUG.TX: now also U401.D2 (PD6); no longer U401.D2 (PD6)
- net USB1_DN renamed USB.DN
- net USB1_DP renamed USB.DP
- net USB2_DN: no longer names the net of U401.U11 (USB_DM2)
- net USB2_DP: no longer names the net of U401.T11 (USB_DP2)
- net WE_N renamed DDR.WE_N
- new net DDR.RST_N: U401.E17 (DDR_RESETN)
- new net ETH.CRS_DV: R405.1
- new net ETH.INT_N: R410.1
- new net ETH.RXD0: R406.1
- new net ETH.RXD1: R407.1
- new net ETH_CRS_DV: R405.2, U401.U8 (PC1)
- new net ETH_INT_N: R410.2, U401.H2 (PI3)
- new net ETH_RXD0: R406.2, U401.U6 (PC4)
- new net ETH_RXD1: R407.2, U401.R7 (PC5)
- new net PMIC.INT_N: U401.G5 (PF8)
- new net PMIC.SCL: U401.D8 (PE15)
- no-connect marks 119 -> 111
Other:
- moved on the sheet: R403, R404
