File: keypad.kicad_sch (KiCad schematic)
At the start: 9 parts, among them J1201 Conn_01x08, U1201 TCA9554PW

Commit message: Add series termination, assign netclasses, fill schemas' descriptions
Parts:
- R1201, R1202: value 1.5 kΩ -> 4.7 kΩ
Changed lines of the file:
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@@
+		)
+	)
+	(text_box "Notes"
+		(exclude_from_sim no)
+		(at 12.7 251.46 0)
+		(size 285.75 33.02)
+		(margins 0.9525 2 0.9525 0.9525)
+		(stroke
+			(width 0)
+			(type solid)
+		)
+		(fill
+			(type none)
+		)
+		(effects
+			(font
+				(size 5.08 5.08)
+				(thickness 1.016)
+				(bold yes)
+			)
+			(justify top)
+		)
+	)
+	(text_box "Keypad interface"
+		(exclude_from_sim no)
+		(at 12.7 50.8 0)
+		(size 393.7 200.66)
+		(margins 0.9525 2 0.9525 0.9525)
+		(stroke
+			(width 0)
+			(type solid)
+		)
+		(fill
+			(type none)
+		)
+		(effects
+			(font
+				(size 5.08 5.08)
+				(thickness 1.016)
+				(bold yes)
+			)
+			(justify top)
+		)
+	)
+	(text_box "They keypad interface is for a 4x4 matrix membrane keypad.\n\nThe keypad buttons are polled continuously and button presses are detected by switching rows and columns HIGH/LOW and changing states between INPUT/OUTPUT.\n\nThe keypad buttons and their usage is application defined and thus not hard-set."
+		(exclude_from_sim no)
+		(at 13.97 63.5 0)
+		(size 391.16 31.75)
+		(margins 0.9525 0.9525 0.9525 0.9525)
+		(stroke
+			(width -0.0001)
+			(type solid)
+		)
+		(fill
+			(type none)
+		)
+		(effects
+			(font
+				(size 2 2)
+			)
+			(justify left top)
 		)
 	)
@@
 			)
 		)
-		(property "Value" "1.5 kΩ"
+		(property "Value" "4.7 kΩ"
 			(at 124.46 132.08 0)
 			(effects
@@
 			)
 		)
-		(property "Value" "1.5 kΩ"
+		(property "Value" "4.7 kΩ"
 			(at 137.16 132.08 0)
 			(effects
