File: user_interface.kicad_sch (KiCad schematic)
At the start: 26 parts, among them J1201 PH1-08-UA, J1202 EMI shield frame, J1203 FH12A-40S-0.5SH(55), U1201 TCA9554PW, U1202 AP5725FDCG-7, X1201 Keypad 3x4, X1202 NHD-4.3-480272EF-ASXP

Commit message: Rework text boxes
Other:
- note added: "Graphical interface"
- note added: "Keypad interface"
- note added: "Notes"
Changed lines of the file:
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@@
+		)
+	)
+	(rectangle
+		(start 209.55 50.8)
+		(end 406.4 251.46)
+		(stroke
+			(width 0)
+			(type default)
+		)
+		(fill
+			(type none)
+		)
+	)
+	(rectangle
+		(start 12.7 251.46)
+		(end 298.45 284.48)
+		(stroke
+			(width 0)
+			(type default)
+		)
+		(fill
+			(type none)
+		)
+	)
+	(rectangle
+		(start 12.7 50.8)
+		(end 209.55 251.46)
+		(stroke
+			(width 0)
+			(type default)
+		)
+		(fill
+			(type none)
 		)
 	)
@@
 			)
 			(justify right)
+		)
+	)
+	(text "Graphical interface"
+		(exclude_from_sim no)
+		(at 210.82 53.34 0)
+		(effects
+			(font
+				(size 5.08 5.08)
+				(thickness 1.016)
+				(bold yes)
+			)
+			(justify left top)
+		)
+	)
+	(text "Keypad interface"
+		(exclude_from_sim no)
+		(at 13.97 53.34 0)
+		(effects
+			(font
+				(size 5.08 5.08)
+				(thickness 1.016)
+				(bold yes)
+			)
+			(justify left top)
 		)
 	)
@@
 				(size 1.27 1.27)
 			)
+		)
+	)
+	(text "Notes"
+		(exclude_from_sim no)
+		(at 13.97 254 0)
+		(effects
+			(font
+				(size 5.08 5.08)
+				(thickness 1.016)
+				(bold yes)
+			)
+			(justify left top)
 		)
 	)
@@
 		)
 	)
-	(text_box "Notes"
-		(exclude_from_sim no)
-		(at 12.7 251.46 0)
-		(size 285.75 33.02)
-		(margins 0.9525 2 0.9525 0.9525)
-		(stroke
-			(width 0)
-			(type solid)
-		)
-		(fill
-			(type none)
-		)
-		(effects
-			(font
-				(size 5.08 5.08)
-				(thickness 1.016)
-				(bold yes)
-			)
-			(justify top)
-		)
-	)
-	(text_box "Keypad interface"
-		(exclude_from_sim no)
-		(at 12.7 50.8 0)
-		(size 196.85 200.66)
-		(margins 0.9525 2 0.9525 0.9525)
-		(stroke
-			(width 0)
-			(type solid)
-		)
-		(fill
-			(type none)
-		)
-		(effects
-			(font
-				(size 5.08 5.08)
-				(thickness 1.016)
-				(bold yes)
-			)
-			(justify top)
-		)
-	)
-	(text_box "Graphical interface"
-		(exclude_from_sim no)
-		(at 209.55 50.8 0)
-		(size 196.85 200.66)
-		(margins 0.9525 2 0.9525 0.9525)
-		(stroke
-			(width 0)
-			(type solid)
-		)
-		(fill
-			(type none)
-		)
-		(effects
-			(font
-				(size 5.08 5.08)
-				(thickness 1.016)
-				(bold yes)
-			)
-			(justify top)
-		)
-	)
