File: user_interface.kicad_sch (KiCad schematic)
At the start: 59 parts, among them J1201 PH1-08-UA, J1202 EMI shield frame, J1203 FH12A-40S-0.5SH(55), U1201 TCA9554PW, U1202 AP5725FDCG-7, X1201 Keypad 3x4, X1202 NHD-4.3-480272EF-ASXP

Commit message: Route the UI section
Connections:
- net INT renamed SCREEN_INT
- net INT_N renamed KEYPAD_INT_N
- net RST renamed SCREEN_RST
- net SCL renamed KEYPAD_SCL
- net KEYPAD_SCL: no longer J1203.39 (Pin_39), R1241.2
- net SDA renamed KEYPAD_SDA
- net KEYPAD_SDA: no longer J1203.40 (Pin_40), R1242.2
- new net SCREEN_SCL: J1203.39 (Pin_39), R1241.2
- new net SCREEN_SDA: J1203.40 (Pin_40), R1242.2
Changed lines of the file:
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@@
 	)
 	(junction
+		(at 330.2 139.7)
+		(diameter 0)
+		(color 0 0 0 0)
+	)
+	(junction
 		(at 95.25 124.46)
 		(diameter 0)
@@
 	)
 	(junction
-		(at 330.2 139.7)
-		(diameter 0)
-		(color 0 0 0 0)
-	)
-	(junction
 		(at 260.35 114.3)
 		(diameter 0)
@@
 	)
 	(label "B6"
-		(at 317.4556 198.12 0)
+		(at 311.1056 198.12 0)
 		(effects
 			(font
@@
 	)
 	(label "G5"
-		(at 317.3559 175.26 0)
+		(at 311.0059 175.26 0)
 		(effects
 			(font
@@
 		)
 	)
-	(label "RST"
-		(at 317.5 223.52 0)
+	(label "SCREEN_RST"
+		(at 311.15 223.52 0)
 		(effects
 			(font
@@
 	)
 	(label "B1"
-		(at 317.5 185.42 0)
+		(at 311.15 185.42 0)
 		(effects
 			(font
@@
 	)
 	(label "HSYNC"
-		(at 317.5 210.82 0)
+		(at 311.15 210.82 0)
 		(effects
 			(font
@@
 	)
 	(label "G7"
-		(at 317.3559 180.34 0)
+		(at 311.0059 180.34 0)
 		(effects
 			(font
@@
 	)
 	(label "G0"
-		(at 317.4833 162.56 0)
+		(at 311.1333 162.56 0)
 		(effects
 			(font
@@
 	)
 	(label "R7"
-		(at 317.4392 160.02 0)
+		(at 311.0892 160.02 0)
 		(effects
 			(font
@@
 	)
 	(label "VSYNC"
-		(at 317.4389 213.36 0)
+		(at 311.0889 213.36 0)
 		(effects
 			(font
@@
 	)
 	(label "B4"
-		(at 317.4556 193.04 0)
+		(at 311.1056 193.04 0)
 		(effects
 			(font
@@
 	)
 	(label "DE"
-		(at 317.4389 215.9 0)
+		(at 311.0889 215.9 0)
 		(effects
 			(font
@@
 	)
 	(label "R5"
-		(at 317.4389 154.94 0)
+		(at 311.0889 154.94 0)
 		(effects
 			(font
@@
 	)
 	(label "R6"
-		(at 317.4389 157.48 0)
+		(at 311.0889 157.48 0)
 		(effects
 			(font
@@
 	)
 	(label "B3"
-		(at 317.5 190.5 0)
+		(at 311.15 190.5 0)
 		(effects
 			(font
@@
 		)
 	)
-	(label "INT"
-		(at 317.5 226.06 0)
+	(label "SCREEN_INT"
+		(at 311.15 226.06 0)
 		(effects
 			(font
@@
 	)
 	(label "R0"
-		(at 317.5 142.24 0)
+		(at 311.15 142.24 0)
 		(effects
 			(font
@@
 		)
 	)
-	(label "SDA"
-		(at 317.5 231.14 0)
+	(label "SCREEN_SDA"
+		(at 311.15 231.14 0)
 		(effects
 			(font
@@
 	)
 	(label "R3"
-		(at 317.5 149.86 0)
+		(at 311.15 149.86 0)
 		(effects
 			(font
@@
 	)
 	(label "G3"
-		(at 317.417 170.18 0)
+		(at 311.067 170.18 0)
 		(effects
 			(font
@@
 		)
 	)
-	(label "SCL"
-		(at 317.5 228.6 0)
+	(label "SCREEN_SCL"
+		(at 311.15 228.6 0)
 		(effects
 			(font
@@
 	)
 	(label "DISP"
-		(at 317.5 208.28 0)
+		(at 311.15 208.28 0)
 		(effects
 			(font
@@
 	)
 	(label "R2"
-		(at 317.5 147.32 0)
+		(at 311.15 147.32 0)
 		(effects
 			(font
@@
 	)
 	(label "G1"
-		(at 317.417 165.1 0)
+		(at 311.067 165.1 0)
 		(effects
 			(font
@@
 	)
 	(label "DCLK"
-		(at 317.5 205.74 0)
+		(at 311.15 205.74 0)
 		(effects
 			(font
@@
 	)
 	(label "B5"
-		(at 317.4556 195.58 0)
+		(at 311.1056 195.58 0)
 		(effects
 			(font
@@
 	)
 	(label "R4"
-		(at 317.5003 152.4 0)
+		(at 311.1503 152.4 0)
 		(effects
 			(font
@@
 		)
 	)
-	(label "INT_N"
-		(at 102.87 124.46 180)
+	(label "KEYPAD_INT_N"
+		(at 80.01 124.46 0)
 		(effects
 			(font
 				(size 1.27 1.27)
 			)
-			(justify right bottom)
+			(justify left bottom)
 		)
 	)
@@
 		)
 	)
-	(label "SCL"
-		(at 102.87 119.38 180)
+	(label "KEYPAD_SCL"
+		(at 80.01 119.38 0)
 		(effects
 			(font
 				(size 1.27 1.27)
 			)
-			(justify right bottom)
+			(justify left bottom)
 		)
 	)
@@
 	)
 	(label "B0"
-		(at 317.5 182.88 0)
+		(at 311.15 182.88 0)
 		(effects
 			(font
@@
 	)
 	(label "B7"
-		(at 317.4556 200.66 0)
+		(at 311.1056 200.66 0)
 		(effects
 			(font
@@
 	)
 	(label "G6"
-		(at 317.4222 177.8 0)
+		(at 311.0722 177.8 0)
 		(effects
 			(font
@@
 	)
 	(label "R1"
-		(at 317.5 144.78 0)
+		(at 311.15 144.78 0)
 		(effects
 			(font
@@
 		)
 	)
-	(label "SDA"
-		(at 102.87 121.92 180)
+	(label "KEYPAD_SDA"
+		(at 80.01 121.92 0)
 		(effects
 			(font
 				(size 1.27 1.27)
 			)
-			(justify right bottom)
+			(justify left bottom)
 		)
 	)
 	(label "G2"
-		(at 317.4833 167.64 0)
+		(at 311.1333 167.64 0)
 		(effects
 			(font
@@
 	)
 	(label "B2"
-		(at 317.5 187.96 0)
+		(at 311.15 187.96 0)
 		(effects
 			(font
@@
 	)
 	(label "G4"
-		(at 317.4222 172.72 0)
+		(at 311.0722 172.72 0)
 		(effects
 			(font

Commit message: Update 0402 footprints
Parts:
- C1205: footprint perfect_footprints:C_0402_1005Metric -> perfect_footprints:C_0402_1005Metric_HDI
